File: MCP39F511_Breakout.kicad_pcb (KiCad board)
At the start: 2 copper layers, 35.6 x 27.9 mm, 28 parts, among them J1 Conn_01x10, U1 MCP39F511-E_MQ, U2 MCP9700T-ETT, Y1 4MHz / 16pF

Commit message: PCB rerouting done
Routing:
- net GND: track 120.6 -> 24.2 mm, vias 27 -> 40
- net VINP: track 38.5 -> 26.8 mm
- net +3V3: track 71.9 -> 83.3 mm, vias 3 -> 2
- net Net-(C4-Pad1): track 21.4 -> 29.7 mm
- net VINN: track 31.9 -> 24.1 mm
- net RX: track 21.6 -> 28.4 mm
- net Net-(TP2-Pad1): track 22.2 -> 28.6 mm
- net Net-(TP1-Pad1): track 24.9 -> 30.8 mm
- net Net-(U1-Pad13): track 11.1 -> 16.6 mm
- net IN: track 14.4 -> 10.3 mm, vias 1 -> 0
- net PWM: track 15.7 -> 17.9 mm
- net Net-(TP3-Pad1): track 8.67 -> 10.7 mm
- net ~RESET: track 15.1 -> 16.9 mm, vias 1 -> 0
- net (no net): track 3.20 -> 2.29 mm
- net IP: track 9.74 -> 10.4 mm
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
Commit message: Create v0.3 board
Routing:
- net GND: track 24.2 -> 24.9 mm
Other:
- board text added: "by Tisham Dhar http://whatnick.com v0.3 11/02/2021"
- board text removed: "by Tisham Dhar http://whatnick.com v0.2 06/12/2020"
Changed lines of the file:
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@@
-(kicad_pcb (version 20201116) (generator pcbnew)
+(kicad_pcb (version 20201220) (generator pcbnew)
   (general
     (thickness 1.6)
@@
     (effects (font (size 1 1) (thickness 0.2)) (justify mirror))
   )
-  (gr_text "by Tisham Dhar\nhttp://whatnick.com\nv0.2 06/12/2020" (at 128.905 94.615) (layer "B.SilkS")
+  (gr_text "by Tisham Dhar\nhttp://whatnick.com\nv0.3 11/02/2021" (at 128.905 94.615) (layer "B.SilkS")
     (effects (font (size 1 1) (thickness 0.25)) (justify mirror))
   )
@@
   (segment (start 141.1 95.4) (end 142.5 96.8) (width 0.25) (layer "B.Cu") (net 12))
   (segment (start 142.8 103) (end 142.8 101.8) (width 0.25) (layer "B.Cu") (net 12))
-  (segment (start 125.3 99.6) (end 125.3 99.5) (width 0.25) (layer "F.Cu") (net 13))
-  (segment (start 125.82 100.1) (end 125.8 100.1) (width 0.25) (layer "F.Cu") (net 13))
-  (segment (start 125.8 100.1) (end 125.3 99.6) (width 0.25) (layer "F.Cu") (net 13))
-  (via (at 125.3 99.5) (size 0.8) (drill 0.4) (layers "F.Cu" "B.Cu") (net 13))
-  (segment (start 128.94999 95.85001) (end 139.95001 95.85001) (width 0.25) (layer "B.Cu") (net 13))
-  (segment (start 128.270001 98.529999) (end 128.270001 96.529999) (width 0.25) (layer "B.Cu") (net 13))
-  (segment (start 141.05 96.95) (end 141.05 103.95) (width 0.25) (layer "B.Cu") (net 13))
-  (segment (start 127.3 99.5) (end 128.270001 98.529999) (width 0.25) (layer "B.Cu") (net 13))
-  (segment (start 141.05 103.95) (end 142.4 105.3) (width 0.25) (layer "B.Cu") (net 13))
-  (segment (start 128.270001 96.529999) (end 128.94999 95.85001) (width 0.25) (layer "B.Cu") (net 13))
-  (segment (start 139.95001 95.85001) (end 141.05 96.95) (width 0.25) (layer "B.Cu") (net 13))
-  (segment (start 125.3 99.5) (end 127.3 99.5) (width 0.25) (layer "B.Cu") (net 13))
+  (segment (start 124.992 100.1) (end 124.46 99.568) (width 0.25) (layer "F.Cu") (net 13))
+  (segment (start 125.82 100.1) (end 124.992 100.1) (width 0.25) (layer "F.Cu") (net 13))
+  (via (at 124.46 99.568) (size 0.8) (drill 0.4) (layers "F.Cu" "B.Cu") (net 13))
+  (segment (start 127.232 99.568) (end 124.46 99.568) (width 0.25) (layer "B.Cu") (net 13))
+  (segment (start 142.4 105.3) (end 141.05 103.95) (width 0.25) (layer "B.Cu") (net 13))
+  (segment (start 141.05 96.95) (end 129.85 96.95) (width 0.25) (layer "B.Cu") (net 13))
+  (segment (start 129.85 96.95) (end 127.232 99.568) (width 0.25) (layer "B.Cu") (net 13))
+  (segment (start 141.05 103.95) (end 141.05 96.95) (width 0.25) (layer "B.Cu") (net 13))
   (segment (start 131.6 106.1) (end 132.1 106.6) (width 0.25) (layer "F.Cu") (net 14))
   (segment (start 130.72 103.493002) (end 131.6 104.373002) (width 0.25) (layer "F.Cu") (net 14))
@@
   (segment (start 139.31 105.41) (end 140.4 106.5) (width 0.25) (layer "F.Cu") (net 17))
   (segment (start 128.27 101.58) (end 129.35 100.5) (width 0.25) (layer "F.Cu") (net 17))
+  (segment (start 127.27 99.15) (end 127.27 98.4598) (width 0.25) (layer "F.Cu") (net 17))
   (segment (start 128.27 101.6) (end 128.3 101.6) (width 0.25) (layer "F.Cu") (net 17))
   (segment (start 127.27 100.27) (end 127.3 100.3) (width 0.25) (layer "F.Cu") (net 17))
